File: mobiflight/stepper_connector.kicad_sch (KiCad schematic)
At the start: 9 parts

Commit message: replace components
Parts:
- renumbered D5 to D2, D6 to D3, D7 to D4, D8 to D5, R5 to R2, R2 to R39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
