File: a320/overhead/lights/a320-overhead-lights/a320-overhead-lights.kicad_pcb (KiCad board)
At the start: 2 copper layers, 77.5 x 107.5 mm, 29 parts, among them J1 Conn_02x11_Odd_Even, J10 Conn_02x08_Odd_Even, J11 Conn_02x08_Odd_Even, J12 Conn_02x08_Odd_Even, J13 Conn_02x08_Odd_Even, J14 Conn_02x08_Odd_Even, J15 Conn_02x08_Odd_Even, J2 Conn_02x08_Odd_Even, J3 Conn_02x03_Odd_Even, J4 Conn_02x08_Odd_Even, J5 Conn_02x08_Odd_Even, J7 Conn_02x08_Odd_Even, J8 Conn_02x09_Odd_Even, J9 Barrel_Jack, U1 LED1642GWPTR, U2 LED1642GWPTR, U3 LED1642GWPTR

Commit message: misc
Parts:
- removed H5: MountingHole, MountingHole:MountingHole_3.2mm_M3
- removed J1: Conn_02x11_Odd_Even, Connector_PinHeader_2.54mm:PinHeader_2x11_P2.54mm_Vertical
- removed J10, J11, J12, J13, J14, J15, J2, J4, J5, J7: Conn_02x08_Odd_Even, Connector_PinHeader_2.54mm:PinHeader_2x08_P2.54mm_Vertical
- removed J3: Conn_02x03_Odd_Even, Connector_PinHeader_2.54mm:PinHeader_2x03_P2.54mm_Vertical
- removed J8: Conn_02x09_Odd_Even, Connector_PinHeader_2.54mm:PinHeader_2x09_P2.54mm_Vertical
- added ANNUN1: SW_SPDT_ON_OFF_ON, Library:ToggleSwitch_MTS-102_SPDT, F.Cu at (263.5, 102.2)
- added APUMASTER1: ~, a320:Korry Switch, F.Cu at (159.7, 105.9)
- added APUSTART1: ~, a320:Korry Switch, F.Cu at (160.0, 135.0)
- added BEACON1: SW_SPDT_ON_ON, Library:ToggleSwitch_MTS-102_SPDT, F.Cu at (58.5, 101.7)
- added D1: LED, LED_THT:LED_D3.0mm, F.Cu at (-87.8, 62.0)
- added D10: LED, LED_THT:LED_D3.0mm, F.Cu at (-81.9, 72.9)
- added D11: LED, LED_THT:LED_D3.0mm, F.Cu at (-81.9, 78.4)
- added D12: LED, LED_THT:LED_D3.0mm, F.Cu at (-81.9, 83.9)
- added D13: LED, LED_THT:LED_D3.0mm, F.Cu at (-81.9, 89.3)
- added D14: LED, LED_THT:LED_D3.0mm, F.Cu at (-81.9, 94.8)
- added D15: LED, LED_THT:LED_D3.0mm, F.Cu at (-76.0, 62.0)
- added D16: LED, LED_THT:LED_D3.0mm, F.Cu at (-76.0, 67.5)
- added D17: LED, LED_THT:LED_D3.0mm, F.Cu at (-76.0, 72.9)
- added D18: LED, LED_THT:LED_D3.0mm, F.Cu at (-76.0, 78.4)
- added D19: LED, LED_THT:LED_D3.0mm, F.Cu at (-76.0, 83.9)
- added D2: LED, LED_THT:LED_D3.0mm, F.Cu at (-87.8, 67.5)
- added D20: LED, LED_THT:LED_D3.0mm, F.Cu at (-76.0, 89.3)
- added D21: LED, LED_THT:LED_D3.0mm, F.Cu at (-76.0, 94.8)
- added D22: LED, LED_THT:LED_D3.0mm, F.Cu at (-70.1, 62.0)
- added D23: LED, LED_THT:LED_D3.0mm, F.Cu at (-70.1, 67.5)
- added D24: LED, LED_THT:LED_D3.0mm, F.Cu at (-70.1, 72.9)
- added D25: LED, LED_THT:LED_D3.0mm, F.Cu at (-70.1, 78.4)
- added D26: LED, LED_THT:LED_D3.0mm, F.Cu at (-70.1, 83.9)
- added D27: LED, LED_THT:LED_D3.0mm, F.Cu at (-70.1, 89.3)
- added D28: LED, LED_THT:LED_D3.0mm, F.Cu at (-70.1, 94.8)
- added D29: LED, LED_THT:LED_D3.0mm, F.Cu at (-64.2, 62.0)
- added D3: LED, LED_THT:LED_D3.0mm, F.Cu at (-87.8, 72.9)
- added D30: LED, LED_THT:LED_D3.0mm, F.Cu at (-64.2, 67.5)
- added D31: LED, LED_THT:LED_D3.0mm, F.Cu at (-64.2, 72.9)
- added D32: LED, LED_THT:LED_D3.0mm, F.Cu at (-64.2, 78.4)
- added D4: LED, LED_THT:LED_D3.0mm, F.Cu at (-87.8, 78.4)
- added D5: LED, LED_THT:LED_D3.0mm, F.Cu at (-87.8, 83.9)
- added D6: LED, LED_THT:LED_D3.0mm, F.Cu at (-87.8, 89.3)
- added D7: LED, LED_THT:LED_D3.0mm, F.Cu at (-87.8, 94.8)
- added D8: LED, LED_THT:LED_D3.0mm, F.Cu at (-81.9, 62.0)
- added D9: LED, LED_THT:LED_D3.0mm, F.Cu at (-81.9, 67.5)
- added DITCHING1: ~, a320:Korry Switch, F.Cu at (262.2, 72.9)
- added DOME1: SW_SPDT_ON_OFF_ON, Library:ToggleSwitch_MTS-102_SPDT, F.Cu at (236.5, 101.7)
- added EMEREXIT1: SW_SPDT_ON_OFF_ON, Library:ToggleSwitch_MTS-102_SPDT, F.Cu at (265.5, 138.3)
- added ENG1AICE1: ~, a320:Korry Switch, F.Cu at (94.7, 44.0)
- added ENG2AICE1: ~, a320:Korry Switch, F.Cu at (122.2, 44.5)
- added ENGEMEREXITLT1: ~, a320:Korry Switch, F.Cu at (232.5, 140.0)
- added INTEGLTPOT1: 10K, Library:Potentiometer_Bourns_PTV09A-1_Single_Vertical, F.Cu at (185.5, 107.5)
- added LANDL1: SW_SPDT_ON_OFF_ON, Library:ToggleSwitch_MTS-102_SPDT, F.Cu at (79.0, 136.8)
- added LANDR1: SW_SPDT_ON_OFF_ON, Library:ToggleSwitch_MTS-102_SPDT, F.Cu at (102.5, 137.2)
- added LDGELEVPOT1: 10K, Library:Potentiometer_Bourns_PTV09A-1_Single_Vertical, F.Cu at (238.1, 70.0)
- added MANVSCTL1: SW_SPDT_(ON)_OFF_(ON), Library:ToggleSwitch_MTS-102_SPDT, F.Cu at (186.0, 65.2)
- added MODESELFAULT1: ~, a320:Korry Switch, F.Cu at (213.5, 63.9)
- added NAV&LOGO1: SW_SPDT_ON_OFF_ON, Library:ToggleSwitch_MTS-102_SPDT, F.Cu at (121.0, 108.5)
- added NOSE1: SW_SPDT_ON_OFF_ON, Library:ToggleSwitch_MTS-102_SPDT, F.Cu at (115.5, 141.5)
- added NOSMOKING1: SW_SPDT_ON_OFF_ON, Library:ToggleSwitch_MTS-102_SPDT, F.Cu at (210.0, 136.8)
- added PROBEWINDOW1: ~, a320:Korry Switch, F.Cu at (149.2, 45.0)
- added RUNWAYTURNOFF1: SW_SPDT_ON_ON, Library:ToggleSwitch_MTS-102_SPDT, F.Cu at (34.5, 135.8)
- added SEATBLTS1: SW_SPDT_ON_ON, Library:ToggleSwitch_MTS-102_SPDT, F.Cu at (186.5, 134.7)
- added STBYCOMPASS1: SW_SPDT_ON_ON, Library:ToggleSwitch_MTS-102_SPDT, F.Cu at (211.0, 105.5)
- added STROBE1: SW_SPDT_ON_OFF_ON, Library:ToggleSwitch_MTS-102_SPDT, F.Cu at (35.5, 100.0)
- added WING1: SW_SPDT_ON_ON, Library:ToggleSwitch_MTS-102_SPDT, F.Cu at (98.5, 104.5)
- added WINGAICE1: ~, a320:Korry Switch, F.Cu at (46.2, 43.5)
- moved R3 271.4 mm to (199.3, -155.6)
- moved R2 259.4 mm to (218.3, -144.5)
- moved C3 258.1 mm to (201.8, -139.0)
- moved C2 243.5 mm to (201.8, -129.0)
- moved J9 243.2 mm to (221.8, -67.7)
- moved R1 240.8 mm to (201.3, -116.6)
- moved C1 223.8 mm to (204.8, -93.5)
- moved A1 203.1 mm to (9.12, -116.5)
- moved U1 152.7 mm to (83.5, -35.8)
- moved U3 151.5 mm to (113.4, -35.3)
- moved U2 150.3 mm to (140.7, -34.5)
- moved H3 149.7 mm to (320.6, 128.3)
- moved H2 149.6 mm to (320.6, 30.0)
- moved H4 103.5 mm to (20.0, 128.3)
- moved H1 88.0 mm to (20.0, 30.0)
Routing:
- net LEDDRV_LATCH: track 131.9 -> 0.00 mm
- net LEDDRV_CLK: track 129.7 -> 0.00 mm
- net +12V: track 110.6 -> 0.00 mm
- net LEDDRV_DATA: track 76.2 -> 0.00 mm
- net ANNUNCIATOR_BRT: track 74.9 -> 0.00 mm
- net BACKLIGHT_BRT: track 68.3 -> 0.00 mm
- net Net-(A1-PadD45): track 24.3 -> 0.00 mm
- net Net-(A1-PadD28): track 24.1 -> 0.00 mm
- net Net-(A1-PadD26): track 23.1 -> 0.00 mm
- net Net-(A1-PadD43): track 23.0 -> 0.00 mm
- net Net-(A1-PadD22): track 22.7 -> 0.00 mm
- net manvsctloff: track 22.5 -> 0.00 mm
- net ditching: track 22.1 -> 0.00 mm
- net apustart: track 21.8 -> 0.00 mm
- net Net-(A1-PadD24): track 21.8 -> 0.00 mm
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- removed copper zone on F.Cu, net +5V
- removed copper zone on B.Cu, net GND
Other:
- board size 77.5 x 107.5 mm -> 308.6 x 106.3 mm
- board text removed: "100nF"
- board text removed: "12V - -(o +"
- board text removed: "12V ->"
- board text removed: "1K"
- board text removed: "5V"
- board text removed: "5V ->"
- board text removed: "<- 5V"
- board text removed: "<- GND"
- board text removed: "A5"
- board text removed: "A6"
- board text removed: "A7"
- board text removed: "BACKLIGHTS 7..0"
- board text removed: "BACKLIGHTS 8..15"
- board text removed: "Backlights 12V"
- board text removed: "D19"
- board text removed: "D22"
- board text removed: "D23"
- board text removed: "D24"
- board text removed: "D25"
- board text removed: "D26"
- board text removed: "D27"
- board text removed: "D28"
- board text removed: "D42"
- board text removed: "D43"
- board text removed: "D44"
- board text removed: "D45"
- board text removed: "D46"
- board text removed: "D47"
- board text removed: "GND"
- board text removed: "GND ->"
- board text removed: "JLCJLCJLCJLC"
- board text removed: "LED 5V"
- board text removed: "annunbrt"
- board text removed: "annunoff"
- board text removed: "apumaster"
- board text removed: "apustart"
- board text removed: "apustarton apustartfault apumasteron apumasterfault modeselon modeselfault probewindowoff probewindowfault"
- board text removed: "beaconon"
- board text removed: "ditching"
- board text removed: "ditchingfault ditchingon emerexitltfault emerexitltoff"
- board text removed: "domebrt"
- board text removed: "domedim"
- board text removed: "emerexitlt"
- board text removed: "emerexitoff"
- board text removed: "emerexiton"
- board text removed: "eng1aice"
- board text removed: "eng2aice"
- board text removed: "integltpot"
- board text removed: "landlon"
- board text removed: "landlretract"
- board text removed: "landron"
- board text removed: "landrretract"
- board text removed: "ldgelevpot"
- board text removed: "manvsctloff"
- board text removed: "manvsctlon"
- board text removed: "modesel"
- board text removed: "nav logo on"
- board text removed: "nav&logooff"
- board text removed: "noseoff"
- board text removed: "noseon"
- board text removed: "nosmokingoff"
- board text removed: "nosmokingon"
- board text removed: "probewindow"
- board text removed: "runwayturnoffon"
- board text removed: "seatbeltson"
- board text removed: "spare"
- board text removed: "stbycompasson"
- board text removed: "strobeoff"
- board text removed: "strobeon"
- board text removed: "wingaice"
- board text removed: "wingaicefault wingaiceon sparefault spareon eng1aicefault eng1aiceon eng2aicefault eng2aiceon"
- board text removed: "wingon"
