File: a320/overhead/lights/a320-overhead-lights/microcontroller.kicad_sch (KiCad schematic)
At the start: 14 parts, among them J1 Conn_02x11_Odd_Even, J2 Conn_02x08_Odd_Even, J3 Conn_02x03_Odd_Even, J4 Conn_02x08_Odd_Even, J5 Conn_02x08_Odd_Even, J6 Conn_02x06_Odd_Even, J7 Conn_02x08_Odd_Even, J8 Conn_02x09_Odd_Even

Commit message: misc
Parts:
- removed H5: MountingHole, MountingHole:MountingHole_3.2mm_M3, symbol Mechanical:MountingHole
