File: a320/overhead/lights/a320-overhead-lights/switches.kicad_sch (KiCad schematic)
At the start: 17 parts

Commit message: misc
Parts:
- ANNUN1, BEACON1, DOME1, EMEREXIT1, LANDL1, LANDR1, MANVSCTL1, NAV&LOGO1, NOSE1, NOSMOKING1, RUNWAYTURNOFF1, SEATBLTS1, STBYCOMPASS1, STROBE1, WING1: footprint (none) -> Library:ToggleSwitch_MTS-102_SPDT
- INTEGLTPOT1, LDGELEVPOT1: footprint (none) -> Library:Potentiometer_Bourns_PTV09A-1_Single_Vertical; symbol Device:R_Potentiometer -> Device:R_Potentiometer_MountingPin
Connections:
- net GND: now also INTEGLTPOT1.MP (MountPin), LDGELEVPOT1.MP (MountPin)
Changed lines of the file:
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@@
 	(generator_version "8.0")
 	(paper "A4")
+	(junction
+		(at 73.66 127)
+		(diameter 0)
+		(color 0 0 0 0)
+	)
+	(junction
+		(at 99.06 127)
+		(diameter 0)
+		(color 0 0 0 0)
+	)
 	(no_connect
 		(at 86.36 22.86)
@@
 	(wire
 		(pts
+			(xy 80.01 121.92) (xy 80.01 119.38)
+		)
+		(stroke
+			(width 0)
+			(type default)
+		)
+	)
+	(wire
+		(pts
 			(xy 73.66 127) (xy 73.66 129.54)
 		)
@@
 	(wire
 		(pts
+			(xy 99.06 119.38) (xy 99.06 127)
+		)
+		(stroke
+			(width 0)
+			(type default)
+		)
+	)
+	(wire
+		(pts
 			(xy 22.86 177.8) (xy 22.86 180.34)
 		)
@@
 	(wire
 		(pts
+			(xy 105.41 119.38) (xy 99.06 119.38)
+		)
+		(stroke
+			(width 0)
+			(type default)
+		)
+	)
+	(wire
+		(pts
+			(xy 80.01 119.38) (xy 73.66 119.38)
+		)
+		(stroke
+			(width 0)
+			(type default)
+		)
+	)
+	(wire
+		(pts
 			(xy 22.86 127) (xy 22.86 129.54)
 		)
@@
 	(wire
 		(pts
+			(xy 105.41 121.92) (xy 105.41 119.38)
+		)
+		(stroke
+			(width 0)
+			(type default)
+		)
+	)
+	(wire
+		(pts
 			(xy 73.66 50.8) (xy 73.66 53.34)
 		)
@@
 	(wire
 		(pts
+			(xy 73.66 119.38) (xy 73.66 127)
+		)
+		(stroke
+			(width 0)
+			(type default)
+		)
+	)
+	(wire
+		(pts
 			(xy 35.56 53.34) (xy 38.1 53.34)
 		)
@@
 	)
 	(symbol
-		(lib_id "Device:R_Potentiometer")
+		(lib_id "Device:R_Potentiometer_MountingPin")
 		(at 80.01 127 90)
 		(mirror x)
@@
 		(exclude_from_sim no)
 		(in_bom yes)
-		(on_board no)
+		(on_board yes)
 		(dnp no)
 		(property "Reference" "INTEGLTPOT1"
@@
 			)
 		)
-		(property "Footprint" ""
+		(property "Footprint" "Library:Potentiometer_Bourns_PTV09A-1_Single_Vertical"
 			(at 80.01 127 0)
 			(effects
@@
 			)
 		)
-		(property "Description" "Potentiometer"
+		(property "Description" "Potentiometer with a mounting pin"
 			(at 80.01 127 0)
 			(effects
@@
 		(pin "3"
 		)
+		(pin "MP"
+		)
 		(instances
 			(project ""
@@
 		(exclude_from_sim no)
 		(in_bom yes)
-		(on_board no)
+		(on_board yes)
 		(dnp no)
 		(fields_autoplaced yes)
@@
 			)
 		)
-		(property "Footprint" ""
+		(property "Footprint" "Library:ToggleSwitch_MTS-102_SPDT"
 			(at 30.48 50.8 0)
 			(effects
@@
 		(exclude_from_sim no)
 		(in_bom yes)
-		(on_board no)
+		(on_board yes)
 		(dnp no)
 		(fields_autoplaced yes)
@@
 			)
 		)
-		(property "Footprint" ""
+		(property "Footprint" "Library:ToggleSwitch_MTS-102_SPDT"
 			(at 30.48 76.2 0)
 			(effects
@@
 		(exclude_from_sim no)
 		(in_bom yes)
-		(on_board no)
+		(on_board yes)
 		(dnp no)
 		(fields_autoplaced yes)
@@
 			)
 		)
-		(property "Footprint" ""
+		(property "Footprint" "Library:ToggleSwitch_MTS-102_SPDT"
 			(at 30.48 152.4 0)
 			(effects
@@
 		(exclude_from_sim no)
 		(in_bom yes)
-		(on_board no)
+		(on_board yes)
 		(dnp no)
 		(fields_autoplaced yes)
@@
 			)
 		)
-		(property "Footprint" ""
+		(property "Footprint" "Library:ToggleSwitch_MTS-102_SPDT"
 			(at 132.08 50.8 0)
 			(effects
@@
 		(exclude_from_sim no)
 		(in_bom yes)
-		(on_board no)
+		(on_board yes)
 		(dnp no)
 		(fields_autoplaced yes)
@@
 			)
 		)
-		(property "Footprint" ""
+		(property "Footprint" "Library:ToggleSwitch_MTS-102_SPDT"
 			(at 30.48 25.4 0)
 			(effects
@@
 		(exclude_from_sim no)
 		(in_bom yes)
-		(on_board no)
+		(on_board yes)
 		(dnp no)
 		(fields_autoplaced yes)
@@
 			)
 		)
-		(property "Footprint" ""
+		(property "Footprint" "Library:ToggleSwitch_MTS-102_SPDT"
 			(at 81.28 25.4 0)
 			(effects
@@
 		(exclude_from_sim no)
 		(in_bom yes)
-		(on_board no)
+		(on_board yes)
 		(dnp no)
 		(fields_autoplaced yes)
@@
 			)
 		)
-		(property "Footprint" ""
+		(property "Footprint" "Library:ToggleSwitch_MTS-102_SPDT"
 			(at 132.08 127 0)
 			(effects
@@
 		(exclude_from_sim no)
 		(in_bom yes)
-		(on_board no)
+		(on_board yes)
 		(dnp no)
 		(fields_autoplaced yes)
@@
 			)
 		)
-		(property "Footprint" ""
+		(property "Footprint" "Library:ToggleSwitch_MTS-102_SPDT"
 			(at 81.28 50.8 0)
 			(effects
@@
 		(exclude_from_sim no)
 		(in_bom yes)
-		(on_board no)
+		(on_board yes)
 		(dnp no)
 		(fields_autoplaced yes)
@@
 			)
 		)
-		(property "Footprint" ""
+		(property "Footprint" "Library:ToggleSwitch_MTS-102_SPDT"
 			(at 81.28 76.2 0)
 			(effects
@@
 	)
 	(symbol
-		(lib_id "Device:R_Potentiometer")
+		(lib_id "Device:R_Potentiometer_MountingPin")
 		(at 105.41 127 90)
 		(mirror x)
@@
 		(exclude_from_sim no)
 		(in_bom yes)
-		(on_board no)
+		(on_board yes)
 		(dnp no)
 		(property "Reference" "LDGELEVPOT1"
@@
 			)
 		)
-		(property "Footprint" ""
+		(property "Footprint" "Library:Potentiometer_Bourns_PTV09A-1_Single_Vertical"
 			(at 105.41 127 0)
 			(effects
@@
 			)
 		)
-		(property "Description" "Potentiometer"
+		(property "Description" "Potentiometer with a mounting pin"
 			(at 105.41 127 0)
 			(effects
@@
 		(pin "3"
 		)
+		(pin "MP"
+		)
 		(instances
 			(project "a320-overhead-lights"
@@
 		(exclude_from_sim no)
 		(in_bom yes)
-		(on_board no)
+		(on_board yes)
 		(dnp no)
 		(fields_autoplaced yes)
@@
 			)
 		)
-		(property "Footprint" ""
+		(property "Footprint" "Library:ToggleSwitch_MTS-102_SPDT"
 			(at 30.48 127 0)
 			(effects
@@
 		(exclude_from_sim no)
 		(in_bom yes)
-		(on_board no)
+		(on_board yes)
 		(dnp no)
 		(fields_autoplaced yes)
@@
 			)
 		)
-		(property "Footprint" ""
+		(property "Footprint" "Library:ToggleSwitch_MTS-102_SPDT"
 			(at 30.48 177.8 0)
 			(effects
@@
 		(exclude_from_sim no)
 		(in_bom yes)
-		(on_board no)
+		(on_board yes)
 		(dnp no)
 		(fields_autoplaced yes)
@@
 			)
 		)
-		(property "Footprint" ""
+		(property "Footprint" "Library:ToggleSwitch_MTS-102_SPDT"
 			(at 132.08 25.4 0)
 			(effects
@@
 		(exclude_from_sim no)
 		(in_bom yes)
-		(on_board no)
+		(on_board yes)
 		(dnp no)
 		(fields_autoplaced yes)
@@
 			)
 		)
-		(property "Footprint" ""
+		(property "Footprint" "Library:ToggleSwitch_MTS-102_SPDT"
 			(at 132.08 76.2 0)
 			(effects
@@
 		(exclude_from_sim no)
 		(in_bom yes)
-		(on_board no)
+		(on_board yes)
 		(dnp no)
 		(fields_autoplaced yes)
@@
 			)
 		)
-		(property "Footprint" ""
+		(property "Footprint" "Library:ToggleSwitch_MTS-102_SPDT"
 			(at 132.08 101.6 0)
 			(effects
@@
 		(exclude_from_sim no)
 		(in_bom yes)
-		(on_board no)
+		(on_board yes)
 		(dnp no)
 		(fields_autoplaced yes)
@@
 			)
 		)
-		(property "Footprint" ""
+		(property "Footprint" "Library:ToggleSwitch_MTS-102_SPDT"
 			(at 30.48 101.6 0)
 			(effects
